File: Eagle/ver 4/ver 3/SCFschem.sch (EAGLE design)
At the start: 9 parts

Commit message: Updated Ribbon Boards and revamped Shield
Parts:
- removed SV6, SV8: (no value), con-lstb:MA05-2
- added H1: STAND-OFF-NEWNEW, SparkFun-Hardware:STAND-OFF-NEWNEW
- added J1, J2: AVR_SPI_PROG_5X2_NEWPTH2, SparkFun-Connectors:AVR_SPI_PROG_5X2_NEWPTH2
Connections:
- net GND: now also J1.GND, J1.GND@1, J1.GND@2, J1.GND@3, J1.GND@4, J2.GND, J2.GND@1, J2.GND@2, J2.GND@3, J2.GND@4; no longer SV6.10, SV6.2, SV6.4, SV6.6, SV6.8, SV8.10, SV8.2, SV8.4, SV8.6, SV8.8
- net S1: now also J1.1; no longer SV6.9
- net S10: now also J2.9; no longer SV8.1
- net S2: now also J1.3; no longer SV6.7
- net S3: now also J1.5; no longer SV6.5
- net S4: now also J1.7; no longer SV6.3
- net S5: now also J1.9; no longer SV6.1
- net S6: now also J2.1; no longer SV8.9
- net S7: now also J2.3; no longer SV8.7
- net S8: now also J2.5; no longer SV8.5
- net S9: now also J2.7; no longer SV8.3
