File: Eagle/Shield/Shield ver 12/shield12.brd (EAGLE design)
At the start: 96 x 75 mm, 42 parts, among them J2 AVR_SPI_PROG_5X2_NEWPTH2, J3 AVR_SPI_PROG_5X2_NEWPTH2, J4 AVR_SPI_PROG_5X2_NEWPTH2, J5 AVR_SPI_PROG_5X2_NEWPTH2, J6 AVR_SPI_PROG_5X2_NEWPTH2, J7 AVR_SPI_PROG_5X2_NEWPTH2, J8 AVR_SPI_PROG_5X2_NEWPTH2, J9 AVR_SPI_PROG_5X2_NEWPTH2

Commit message: Added pins 51 and 52 to use SPI for LEDS, re ran gerbers. The code now outputs to the LEDS over SPI and edits were made so that the strip is only outputted once
Parts:
- removed OPAMP1:RN1, OPAMP1:RN2, OPAMP1:RN3, OPAMP1:RN4, OPAMP2:RN1, OPAMP2:RN2, OPAMP2:RN3, OPAMP2:RN4, OPAMP3:RN1, OPAMP3:RN2, OPAMP3:RN3, OPAMP3:RN4, OPAMP4:RN1, OPAMP4:RN2, OPAMP4:RN3, OPAMP4:RN4, OPAMP5:RN1, OPAMP5:RN2, OPAMP5:RN3, OPAMP5:RN4: 10k, SparkFun-Resistors:0805-ARV_EDIT10K
- added OPAMP1:R1, OPAMP1:R2, OPAMP1:R3, OPAMP1:R4, OPAMP2:R1, OPAMP2:R2, OPAMP2:R3, OPAMP2:R4, OPAMP3:R1, OPAMP3:R2, OPAMP3:R3, OPAMP3:R4, OPAMP4:R1, OPAMP4:R2, OPAMP4:R3, OPAMP4:R4, OPAMP5:R1, OPAMP5:R2, OPAMP5:R3, OPAMP5:R4: YC164-JR-0710KL, YC164 Resistor Array:YAG_YC164
- B2: value ARDUINO_MEGA_R3_EDITARDUINO_MEGA_EDIT -> ARDUINO_MEGA_R3_EDIT
- moved X10 4.02 mm to (91.4, 50.8)
- moved X11 4.02 mm to (91.4, 30.5)
Connections:
- net A10O: now also OPAMP5:R4.5, OPAMP5:R4.6, OPAMP5:R4.7, OPAMP5:R4.8; no longer OPAMP5:RN4.5, OPAMP5:RN4.6, OPAMP5:RN4.7, OPAMP5:RN4.8
- net A1O: now also OPAMP1:R2.5, OPAMP1:R2.6, OPAMP1:R2.7, OPAMP1:R2.8; no longer OPAMP1:RN2.5, OPAMP1:RN2.6, OPAMP1:RN2.7, OPAMP1:RN2.8
- net A2O: now also OPAMP2:R2.5, OPAMP2:R2.6, OPAMP2:R2.7, OPAMP2:R2.8; no longer OPAMP2:RN2.5, OPAMP2:RN2.6, OPAMP2:RN2.7, OPAMP2:RN2.8
- net A3O: now also OPAMP3:R2.5, OPAMP3:R2.6, OPAMP3:R2.7, OPAMP3:R2.8; no longer OPAMP3:RN2.5, OPAMP3:RN2.6, OPAMP3:RN2.7, OPAMP3:RN2.8
- net A4O: now also OPAMP4:R2.5, OPAMP4:R2.6, OPAMP4:R2.7, OPAMP4:R2.8; no longer OPAMP4:RN2.5, OPAMP4:RN2.6, OPAMP4:RN2.7, OPAMP4:RN2.8
- net A5O: now also OPAMP5:R2.5, OPAMP5:R2.6, OPAMP5:R2.7, OPAMP5:R2.8; no longer OPAMP5:RN2.5, OPAMP5:RN2.6, OPAMP5:RN2.7, OPAMP5:RN2.8
- net A6O: now also OPAMP1:R4.5, OPAMP1:R4.6, OPAMP1:R4.7, OPAMP1:R4.8; no longer OPAMP1:RN4.5, OPAMP1:RN4.6, OPAMP1:RN4.7, OPAMP1:RN4.8
- net A7O: now also OPAMP2:R4.5, OPAMP2:R4.6, OPAMP2:R4.7, OPAMP2:R4.8; no longer OPAMP2:RN4.5, OPAMP2:RN4.6, OPAMP2:RN4.7, OPAMP2:RN4.8
- net A8O: now also OPAMP3:R4.5, OPAMP3:R4.6, OPAMP3:R4.7, OPAMP3:R4.8; no longer OPAMP3:RN4.5, OPAMP3:RN4.6, OPAMP3:RN4.7, OPAMP3:RN4.8
- net A9O: now also OPAMP4:R4.5, OPAMP4:R4.6, OPAMP4:R4.7, OPAMP4:R4.8; no longer OPAMP4:RN4.5, OPAMP4:RN4.6, OPAMP4:RN4.7, OPAMP4:RN4.8
- net OPAMP1:N$1: now also OPAMP1:R3.5, OPAMP1:R3.6, OPAMP1:R3.7, OPAMP1:R3.8, OPAMP1:R4.1, OPAMP1:R4.2, OPAMP1:R4.3, OPAMP1:R4.4; no longer OPAMP1:RN3.5, OPAMP1:RN3.6, OPAMP1:RN3.7, OPAMP1:RN3.8, OPAMP1:RN4.1, OPAMP1:RN4.2, OPAMP1:RN4.3, OPAMP1:RN4.4
- net OPAMP1:N$2: now also OPAMP1:R1.5, OPAMP1:R1.6, OPAMP1:R1.7, OPAMP1:R1.8, OPAMP1:R2.1, OPAMP1:R2.2, OPAMP1:R2.3, OPAMP1:R2.4; no longer OPAMP1:RN1.5, OPAMP1:RN1.6, OPAMP1:RN1.7, OPAMP1:RN1.8, OPAMP1:RN2.1, OPAMP1:RN2.2, OPAMP1:RN2.3, OPAMP1:RN2.4
- net OPAMP2:N$1: now also OPAMP2:R3.5, OPAMP2:R3.6, OPAMP2:R3.7, OPAMP2:R3.8, OPAMP2:R4.1, OPAMP2:R4.2, OPAMP2:R4.3, OPAMP2:R4.4; no longer OPAMP2:RN3.5, OPAMP2:RN3.6, OPAMP2:RN3.7, OPAMP2:RN3.8, OPAMP2:RN4.1, OPAMP2:RN4.2, OPAMP2:RN4.3, OPAMP2:RN4.4
- net OPAMP2:N$2: now also OPAMP2:R1.5, OPAMP2:R1.6, OPAMP2:R1.7, OPAMP2:R1.8, OPAMP2:R2.1, OPAMP2:R2.2, OPAMP2:R2.3, OPAMP2:R2.4; no longer OPAMP2:RN1.5, OPAMP2:RN1.6, OPAMP2:RN1.7, OPAMP2:RN1.8, OPAMP2:RN2.1, OPAMP2:RN2.2, OPAMP2:RN2.3, OPAMP2:RN2.4
- net OPAMP3:N$1: now also OPAMP3:R3.5, OPAMP3:R3.6, OPAMP3:R3.7, OPAMP3:R3.8, OPAMP3:R4.1, OPAMP3:R4.2, OPAMP3:R4.3, OPAMP3:R4.4; no longer OPAMP3:RN3.5, OPAMP3:RN3.6, OPAMP3:RN3.7, OPAMP3:RN3.8, OPAMP3:RN4.1, OPAMP3:RN4.2, OPAMP3:RN4.3, OPAMP3:RN4.4
- net OPAMP3:N$2: now also OPAMP3:R1.5, OPAMP3:R1.6, OPAMP3:R1.7, OPAMP3:R1.8, OPAMP3:R2.1, OPAMP3:R2.2, OPAMP3:R2.3, OPAMP3:R2.4; no longer OPAMP3:RN1.5, OPAMP3:RN1.6, OPAMP3:RN1.7, OPAMP3:RN1.8, OPAMP3:RN2.1, OPAMP3:RN2.2, OPAMP3:RN2.3, OPAMP3:RN2.4
- net OPAMP4:N$1: now also OPAMP4:R3.5, OPAMP4:R3.6, OPAMP4:R3.7, OPAMP4:R3.8, OPAMP4:R4.1, OPAMP4:R4.2, OPAMP4:R4.3, OPAMP4:R4.4; no longer OPAMP4:RN3.5, OPAMP4:RN3.6, OPAMP4:RN3.7, OPAMP4:RN3.8, OPAMP4:RN4.1, OPAMP4:RN4.2, OPAMP4:RN4.3, OPAMP4:RN4.4
- net OPAMP4:N$2: now also OPAMP4:R1.5, OPAMP4:R1.6, OPAMP4:R1.7, OPAMP4:R1.8, OPAMP4:R2.1, OPAMP4:R2.2, OPAMP4:R2.3, OPAMP4:R2.4; no longer OPAMP4:RN1.5, OPAMP4:RN1.6, OPAMP4:RN1.7, OPAMP4:RN1.8, OPAMP4:RN2.1, OPAMP4:RN2.2, OPAMP4:RN2.3, OPAMP4:RN2.4
- net OPAMP5:N$1: now also OPAMP5:R3.5, OPAMP5:R3.6, OPAMP5:R3.7, OPAMP5:R3.8, OPAMP5:R4.1, OPAMP5:R4.2, OPAMP5:R4.3, OPAMP5:R4.4; no longer OPAMP5:RN3.5, OPAMP5:RN3.6, OPAMP5:RN3.7, OPAMP5:RN3.8, OPAMP5:RN4.1, OPAMP5:RN4.2, OPAMP5:RN4.3, OPAMP5:RN4.4
- net OPAMP5:N$2: now also OPAMP5:R1.5, OPAMP5:R1.6, OPAMP5:R1.7, OPAMP5:R1.8, OPAMP5:R2.1, OPAMP5:R2.2, OPAMP5:R2.3, OPAMP5:R2.4; no longer OPAMP5:RN1.5, OPAMP5:RN1.6, OPAMP5:RN1.7, OPAMP5:RN1.8, OPAMP5:RN2.1, OPAMP5:RN2.2, OPAMP5:RN2.3, OPAMP5:RN2.4
- net S10A: no longer OPAMP5:RN1.2
- net S10B: now also OPAMP5:R3.2; no longer OPAMP5:RN3.3
- net S11A: no longer OPAMP1:RN1.3
- net S11B: now also OPAMP1:R3.3; no longer OPAMP1:RN3.2
- net S12A: no longer OPAMP2:RN1.3
- net S12B: now also OPAMP2:R3.3; no longer OPAMP2:RN3.2
- net S13A: no longer OPAMP3:RN1.3
- net S13B: now also OPAMP3:R3.3; no longer OPAMP3:RN3.2
- net S14A: no longer OPAMP4:RN1.3
- net S14B: now also OPAMP4:R3.3; no longer OPAMP4:RN3.2
- net S15A: no longer OPAMP5:RN1.3
- net S15B: now also OPAMP5:R3.3; no longer OPAMP5:RN3.2
- net S16A: no longer OPAMP1:RN1.4
- net S16B: now also OPAMP1:R3.4; no longer OPAMP1:RN3.1
- net S17A: no longer OPAMP2:RN1.4
- net S17B: now also OPAMP2:R3.4; no longer OPAMP2:RN3.1
- net S18A: no longer OPAMP3:RN1.4
- net S18B: now also OPAMP3:R3.4; no longer OPAMP3:RN3.1
- net S19A: no longer OPAMP4:RN1.4
- net S19B: now also OPAMP4:R3.4; no longer OPAMP4:RN3.1
- net S1A: no longer OPAMP1:RN1.1
- net S1B: now also OPAMP1:R3.1; no longer OPAMP1:RN3.4
- net S20A: no longer OPAMP5:RN1.4
- net S20B: now also OPAMP5:R3.4; no longer OPAMP5:RN3.1
- net S2A: no longer OPAMP2:RN1.1
- net S2B: now also OPAMP2:R3.1; no longer OPAMP2:RN3.4
- net S3A: no longer OPAMP3:RN1.1
- net S3B: now also OPAMP3:R3.1; no longer OPAMP3:RN3.4
- net S4A: no longer OPAMP4:RN1.1
- net S4B: now also OPAMP4:R3.1; no longer OPAMP4:RN3.4
- net S5A: no longer OPAMP5:RN1.1
- net S5B: now also OPAMP5:R3.1; no longer OPAMP5:RN3.4
- net S6A: no longer OPAMP1:RN1.2
- net S6B: now also OPAMP1:R3.2; no longer OPAMP1:RN3.3
- net S7A: no longer OPAMP2:RN1.2
- net S7B: now also OPAMP2:R3.2; no longer OPAMP2:RN3.3
- net S8A: no longer OPAMP3:RN1.2
- net S8B: now also OPAMP3:R3.2; no longer OPAMP3:RN3.3
- net S9A: no longer OPAMP4:RN1.2
- net S9B: now also OPAMP4:R3.2; no longer OPAMP4:RN3.3
Routing:
- net S1B: track 118.6 -> 0.00 mm, vias 1 -> 0
- net S6B: track 78.6 -> 0.00 mm, vias 2 -> 0
- net S11B: track 53.2 -> 0.00 mm, vias 1 -> 0
- net S7A: track 35.4 -> 0.00 mm, vias 1 -> 0
- net S20A: track 95.0 -> 73.9 mm
- net S13B: track 74.0 -> 57.9 mm
- net OPAMP1:N$1: track 16.0 -> 0.00 mm
- net OPAMP2:N$1: track 15.6 -> 0.00 mm
- net OPAMP2:N$2: track 15.4 -> 0.00 mm
- net OPAMP3:N$2: track 14.8 -> 0.00 mm
- net OPAMP5:N$2: track 14.5 -> 0.00 mm
- net OPAMP4:N$2: track 14.4 -> 0.00 mm
- net OPAMP1:N$2: track 14.4 -> 0.00 mm
- net OPAMP5:N$1: track 14.3 -> 0.00 mm
- net OPAMP4:N$1: track 14.3 -> 0.00 mm
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